File: pcb/MOKETA.kicad_pcb (KiCad board)
At the start: 2 copper layers, 285 x 114.5 mm, 42 parts

Commit message: New MOKETA otuline
Parts:
- moved SW35 6.32 mm to (259.0, 152.0)
- moved SW22 6.32 mm to (266.3, 105.7)
- moved SW24 6.32 mm to (285.9, 105.3)
- moved SW28 6.32 mm to (326.4, 109.3)
- moved SW29 6.32 mm to (254.1, 133.6)
- moved SW31 6.32 mm to (237.5, 145.3)
- moved SW32 6.32 mm to (311.1, 125.6)
- moved SW34 6.32 mm to (331.4, 127.7)
- moved SW38 6.32 mm to (316.0, 144.0)
- moved SW39 6.32 mm to (336.3, 146.1)
- moved SW40 6.32 mm to (263.9, 170.4)
- moved SW41 6.32 mm to (247.4, 182.1)
- moved SW23 6.32 mm to (249.1, 115.2)
- moved SW25 6.32 mm to (232.6, 126.9)
- moved SW37 6.32 mm to (242.4, 163.7)
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Other:
- board size 285 x 114.5 mm -> 279.6 x 107.1 mm

Commit message: aling col and row
Parts:
- added D1: Diode, moketa:D_SOD-323, F.Cu at (199.2, 142.8)
- added D10: Diode, moketa:D_SOD-323, F.Cu at (203.5, 148.7)
- added D11: Diode, moketa:D_SOD-323, F.Cu at (203.5, 151.7)
- added D12: Diode, moketa:D_SOD-323, F.Cu at (203.5, 154.6)
- added D13: Diode, moketa:D_SOD-323, F.Cu at (203.5, 157.6)
- added D14: Diode, moketa:D_SOD-323, F.Cu at (203.5, 160.5)
- added D15: Diode, moketa:D_SOD-323, F.Cu at (207.8, 142.8)
- added D16: Diode, moketa:D_SOD-323, F.Cu at (207.8, 145.8)
- added D17: Diode, moketa:D_SOD-323, F.Cu at (207.8, 148.7)
- added D18: Diode, moketa:D_SOD-323, F.Cu at (207.8, 151.7)
- added D19: Diode, moketa:D_SOD-323, F.Cu at (207.8, 154.6)
- added D2: Diode, moketa:D_SOD-323, F.Cu at (199.2, 145.8)
- added D20: Diode, moketa:D_SOD-323, F.Cu at (207.8, 157.6)
- added D21: Diode, moketa:D_SOD-323, F.Cu at (207.8, 160.5)
- added D22: Diode, moketa:D_SOD-323, F.Cu at (212.1, 142.8)
- added D23: Diode, moketa:D_SOD-323, F.Cu at (212.1, 145.8)
- added D24: Diode, moketa:D_SOD-323, F.Cu at (212.1, 148.7)
- added D25: Diode, moketa:D_SOD-323, F.Cu at (212.1, 151.7)
- added D26: Diode, moketa:D_SOD-323, F.Cu at (212.1, 154.6)
- added D27: Diode, moketa:D_SOD-323, F.Cu at (212.1, 157.6)
- added D28: Diode, moketa:D_SOD-323, F.Cu at (212.1, 160.5)
- added D29: Diode, moketa:D_SOD-323, F.Cu at (216.4, 142.8)
- added D3: Diode, moketa:D_SOD-323, F.Cu at (199.2, 148.7)
- added D30: Diode, moketa:D_SOD-323, F.Cu at (216.4, 145.8)
- added D31: Diode, moketa:D_SOD-323, F.Cu at (216.4, 148.7)
- added D32: Diode, moketa:D_SOD-323, F.Cu at (216.4, 151.7)
- added D33: Diode, moketa:D_SOD-323, F.Cu at (216.4, 154.6)
- added D34: Diode, moketa:D_SOD-323, F.Cu at (216.4, 157.6)
- added D35: Diode, moketa:D_SOD-323, F.Cu at (216.4, 160.5)
- added D36: Diode, moketa:D_SOD-323, F.Cu at (220.7, 142.8)
- added D37: Diode, moketa:D_SOD-323, F.Cu at (220.7, 145.8)
- added D38: Diode, moketa:D_SOD-323, F.Cu at (220.7, 148.7)
- added D39: Diode, moketa:D_SOD-323, F.Cu at (220.7, 151.7)
- added D4: Diode, moketa:D_SOD-323, F.Cu at (199.2, 151.7)
- added D40: Diode, moketa:D_SOD-323, F.Cu at (220.7, 154.6)
- added D41: Diode, moketa:D_SOD-323, F.Cu at (220.7, 157.6)
- added D42: Diode, moketa:D_SOD-323, F.Cu at (220.7, 160.5)
- added D5: Diode, moketa:D_SOD-323, F.Cu at (199.2, 154.6)
- added D6: Diode, moketa:D_SOD-323, F.Cu at (199.2, 157.6)
- added D7: Diode, moketa:D_SOD-323, F.Cu at (199.2, 160.5)
- added D8: Diode, moketa:D_SOD-323, F.Cu at (203.5, 142.8)
- added D9: Diode, moketa:D_SOD-323, F.Cu at (203.5, 145.8)
- added U1: Pro_Micro, moketa:U_PRO_MICRO, F.Cu at (210.1, 108.8)
- SW1, SW10, SW11, SW12, SW13, SW14, SW15, SW16, SW17, SW18, SW19, SW2, SW20, SW21, SW22, SW23, SW24, SW25, SW26, SW27, SW28, SW29, SW3, SW30, SW31, SW32, SW33, SW34, SW35, SW36, SW37, SW38, SW39, SW4, SW40, SW41, SW42, SW5, SW6, SW7, SW8, SW9: footprint moketa:Kailh_socket_MX -> moketa:SW_PUSH
- moved SW12 239.5 mm to (326.4, 109.3), turned to 15 degrees
- moved SW26 206.5 mm to (103.0, 144.0), turned to -15 degrees
- moved SW28 186.6 mm to (142.8, 142.5), turned to -15 degrees
- moved SW10 179.2 mm to (285.9, 105.3), turned to 15 degrees
- moved SW25 151.1 mm to (82.7, 146.1), turned to -15 degrees
- moved SW27 149.1 mm to (123.2, 142.1), turned to -15 degrees
- moved SW11 130.4 mm to (306.2, 107.2), turned to 15 degrees
- moved SW8 121.3 mm to (249.1, 115.2), turned to 15 degrees
- moved SW30 121.1 mm to (176.6, 163.7), turned to -15 degrees
- moved SW40 108.9 mm to (155.1, 170.4), turned to -15 degrees
- moved SW9 105.2 mm to (266.3, 105.7), turned to 15 degrees
- moved SW21 104.7 mm to (271.2, 124.1), turned to 15 degrees
- moved SW18 98.8 mm to (181.5, 145.3)
- moved SW29 95.9 mm to (160.0, 152.0), turned to -15 degrees
- moved SW20 95.7 mm to (254.1, 133.6), turned to 15 degrees
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Connections:
- SW1 pad 1: Net-(SW1-Pad1) -> COL0
- SW10 pad 1: Net-(SW10-Pad1) -> COL3
- SW11 pad 1: Net-(SW11-Pad1) -> COL4
- SW12 pad 1: Net-(SW12-Pad1) -> COL5
- SW13 pad 1: Net-(SW13-Pad1) -> COL0
- SW14 pad 1: Net-(SW14-Pad1) -> COL1
- SW15 pad 1: Net-(SW1-Pad1) -> COL2
- SW16 pad 1: Net-(SW1-Pad1) -> COL3
- SW17 pad 1: Net-(SW17-Pad1) -> COL4
- SW18 pad 1: Net-(SW17-Pad1) -> COL5
- SW19 pad 1: Net-(SW10-Pad1) -> COL0
- SW2 pad 1: Net-(SW17-Pad1) -> COL1
- SW20 pad 1: Net-(SW10-Pad1) -> COL1
- SW21 pad 1: Net-(SW11-Pad1) -> COL2
- SW22 pad 1: Net-(SW11-Pad1) -> COL3
- SW23 pad 1: Net-(SW12-Pad1) -> COL4
- SW24 pad 1: Net-(SW12-Pad1) -> COL5
- SW25 pad 1: Net-(SW13-Pad1) -> COL0
- SW26 pad 1: Net-(SW13-Pad1) -> COL1
- SW27 pad 1: Net-(SW14-Pad1) -> COL2
- SW28 pad 1: Net-(SW14-Pad1) -> COL3
- SW29 pad 1: Net-(SW1-Pad1) -> COL4
- SW3 pad 1: Net-(SW10-Pad1) -> COL2
- SW30 pad 1: Net-(SW1-Pad1) -> COL5
- SW31 pad 1: Net-(SW17-Pad1) -> COL0
- SW32 pad 1: Net-(SW17-Pad1) -> COL1
- SW33 pad 1: Net-(SW10-Pad1) -> COL2
- SW34 pad 1: Net-(SW10-Pad1) -> COL3
- SW35 pad 1: Net-(SW11-Pad1) -> COL4
- SW36 pad 1: Net-(SW11-Pad1) -> COL5
- SW37 pad 1: Net-(SW12-Pad1) -> COL0
- SW38 pad 1: Net-(SW12-Pad1) -> COL1
- SW39 pad 1: Net-(SW13-Pad1) -> COL2
- SW4 pad 1: Net-(SW11-Pad1) -> COL3
- SW40 pad 1: Net-(SW13-Pad1) -> COL3
- SW41 pad 1: Net-(SW14-Pad1) -> COL4
- SW42 pad 1: Net-(SW14-Pad1) -> COL5
- SW5 pad 1: Net-(SW12-Pad1) -> COL4
- SW6 pad 1: Net-(SW13-Pad1) -> COL5
- SW7 pad 1: Net-(SW14-Pad1) -> COL0
- SW8 pad 1: Net-(SW1-Pad1) -> COL1
- SW9 pad 1: Net-(SW17-Pad1) -> COL2
Routing:
- net Net-(SW11-Pad1): track 48.5 -> 0.00 mm
- net Net-(SW10-Pad1): track 22.0 -> 0.00 mm

Commit message: add footrpint
Parts:
- added LED**: YS-SK6812MINI-E, moketa:YS-SK6812MINI-E, F.Cu at (90.5, 114.8)
- D1, D10, D11, D12, D13, D14, D15, D16, D17, D18, D19, D2, D20, D21, D22, D23, D24, D25, D26, D27, D28, D29, D3, D30, D31, D32, D33, D34, D35, D36, D37, D38, D39, D4, D40, D41, D42, D5, D6, D7, D8, D9: footprint moketa:D_SOD-323 -> moketa:D_SOD-123
- moved D1 119.2 mm to (84.0, 112.3), turned to 75 degrees
- moved D2 101.4 mm to (104.3, 110.3), turned to 75 degrees
- moved D8 44.8 mm to (243.3, 122.1), turned to 105 degrees
