File: pcb/MOKETA.kicad_pcb (KiCad board)
At the start: 2 copper layers, 279.6 x 107.1 mm, 86 parts, among them U1 Pro_Micro

Commit message: update footprint
Parts:
- removed LED**: YS-SK6812MINI-E, moketa:YS-SK6812MINI-E
- moved SW12 230.2 mm to (109.1, 185.0), turned to 0 degrees
- moved SW11 205.4 mm to (109.1, 164.9), turned to 0 degrees
- moved SW24 190.9 mm to (149.3, 185.0), turned to 0 degrees
- moved SW10 181.2 mm to (109.1, 144.8), turned to 0 degrees
- moved D8 173.3 mm to (100.7, 220.6), turned to 0 degrees
- moved SW23 166.6 mm to (149.3, 164.9), turned to 0 degrees
- moved U1 160.0 mm to (88.4, 212.5)
- moved SW9 158.4 mm to (109.1, 124.7), turned to 0 degrees
- moved SW36 151.9 mm to (189.5, 185.0), turned to 0 degrees
- moved SW22 143.2 mm to (149.3, 144.8), turned to 0 degrees
- moved SW8 140.5 mm to (109.1, 104.6), turned to 0 degrees
- moved D36 130.8 mm to (118.1, 224.0)
- moved SW7 130.6 mm to (109.1, 84.5), turned to 0 degrees
- moved D9 129.2 mm to (100.7, 224.0)
- moved SW35 128.3 mm to (189.5, 164.9), turned to 0 degrees
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Connections:
- D1 pad 1: ROW0 -> R0
- D10 pad 1: ROW1 -> R1
- D11 pad 1: ROW1 -> R1
- D12 pad 1: ROW1 -> R1
- D13 pad 1: ROW2 -> R2
- D14 pad 1: ROW2 -> R2
- D15 pad 1: ROW2 -> R2
- D16 pad 1: ROW2 -> R2
- D17 pad 1: ROW2 -> R2
- D18 pad 1: ROW2 -> R2
- D19 pad 1: ROW3 -> R3
- D2 pad 1: ROW0 -> R0
- D20 pad 1: ROW3 -> R3
- D21 pad 1: ROW3 -> R3
- D22 pad 1: ROW3 -> R3
- D23 pad 1: ROW3 -> R3
- D24 pad 1: ROW3 -> R3
- D25 pad 1: ROW4 -> R4
- D26 pad 1: ROW4 -> R4
- D27 pad 1: ROW4 -> R4
- D28 pad 1: ROW4 -> R4
- D29 pad 1: ROW4 -> R4
- D3 pad 1: ROW0 -> R0
- D30 pad 1: ROW4 -> R4
- D31 pad 1: ROW5 -> R5
- D32 pad 1: ROW5 -> R5
- D33 pad 1: ROW5 -> R5
- D34 pad 1: ROW5 -> R5
- D35 pad 1: ROW5 -> R5
- D36 pad 1: ROW5 -> R5
- D37 pad 1: ROW6 -> R6
- D38 pad 1: ROW6 -> R6
- D39 pad 1: ROW6 -> R6
- D4 pad 1: ROW0 -> R0
- D40 pad 1: ROW6 -> R6
- D41 pad 1: ROW6 -> R6
- D42 pad 1: ROW6 -> R6
- D5 pad 1: ROW0 -> R0
- D6 pad 1: ROW0 -> R0
- D7 pad 1: ROW1 -> R1
- D8 pad 1: ROW1 -> R1
- D9 pad 1: ROW1 -> R1
- SW1 pad 1: COL0 -> C0
- SW10 pad 1: COL3 -> C3
- SW11 pad 1: COL4 -> C4
- SW12 pad 1: COL5 -> C5
- SW13 pad 1: COL0 -> C0
- SW14 pad 1: COL1 -> C1
- SW15 pad 1: COL2 -> C2
- SW16 pad 1: COL3 -> C3
- SW17 pad 1: COL4 -> C4
- SW18 pad 1: COL5 -> C5
- SW19 pad 1: COL0 -> C0
- SW2 pad 1: COL1 -> C1
- SW20 pad 1: COL1 -> C1
- SW21 pad 1: COL2 -> C2
- SW22 pad 1: COL3 -> C3
- SW23 pad 1: COL4 -> C4
- SW24 pad 1: COL5 -> C5
- SW25 pad 1: COL0 -> C0
- SW26 pad 1: COL1 -> C1
- SW27 pad 1: COL2 -> C2
- SW28 pad 1: COL3 -> C3
- SW29 pad 1: COL4 -> C4
- SW3 pad 1: COL2 -> C2
- SW30 pad 1: COL5 -> C5
- SW31 pad 1: COL0 -> C0
- SW32 pad 1: COL1 -> C1
- SW33 pad 1: COL2 -> C2
- SW34 pad 1: COL3 -> C3
- SW35 pad 1: COL4 -> C4
- SW36 pad 1: COL5 -> C5
- SW37 pad 1: COL0 -> C3
- SW38 pad 1: COL1 -> C4
- SW39 pad 1: COL2 -> C5
- SW4 pad 1: COL3 -> C3
- SW40 pad 1: COL3 -> C0
- SW41 pad 1: COL4 -> C1
- SW42 pad 1: COL5 -> C2
- SW5 pad 1: COL4 -> C4
- SW6 pad 1: COL5 -> C5
- SW7 pad 1: COL0 -> C0
- SW8 pad 1: COL1 -> C1
- SW9 pad 1: COL2 -> C2
- U1 pad 10: unconnected-(U1-7/E6-Pad10) -> C2
- U1 pad 13: unconnected-(U1-B6/10-Pad13) -> R6
- U1 pad 15: unconnected-(U1-B3/14-Pad15) -> C5
- U1 pad 16: unconnected-(U1-B1/15-Pad16) -> C4
- U1 pad 17: unconnected-(U1-F7/A0-Pad17) -> C3
- U1 pad 18: unconnected-(U1-F6/A1-Pad18) -> R5
- U1 pad 19: unconnected-(U1-F5/A2-Pad19) -> R3
- U1 pad 20: unconnected-(U1-F4/A3-Pad20) -> R1
- U1 pad 22: unconnected-(U1-RST-Pad22) -> RST
- U1 pad 23: unconnected-(U1-GND-Pad23) -> GND
- U1 pad 24: unconnected-(U1-RAW-Pad24) -> VBUS
- U1 pad 3: unconnected-(U1-GND-Pad3) -> GND
- U1 pad 4: unconnected-(U1-GND-Pad4) -> GND
- U1 pad 5: unconnected-(U1-2/D1/SDA-Pad5) -> R0
- U1 pad 6: unconnected-(U1-3/D0/SCL-Pad6) -> R2
- U1 pad 7: unconnected-(U1-4/D4-Pad7) -> R4
- U1 pad 8: unconnected-(U1-5/C6-Pad8) -> C0
- U1 pad 9: unconnected-(U1-6/D7-Pad9) -> C1
Other:
- board outline removed

Commit message: some fix
Parts:
- removed D1, D10, D11, D12, D13, D14, D15, D16, D17, D18, D19, D2, D20, D21, D22, D23, D24, D25, D26, D27, D28, D29, D3, D30, D31, D32, D33, D34, D35, D36, D37, D38, D39, D4, D40, D41, D42, D5, D6, D7, D8, D9: Diode, moketa:D_SOD-123
- removed SW1, SW10, SW11, SW12, SW13, SW14, SW15, SW16, SW17, SW18, SW19, SW2, SW20, SW21, SW22, SW23, SW24, SW25, SW26, SW27, SW28, SW29, SW3, SW30, SW31, SW32, SW33, SW34, SW35, SW36, SW37, SW38, SW39, SW4, SW40, SW41, SW42, SW5, SW6, SW7, SW8, SW9: ~, moketa:SW_PUSH
- removed U1: Pro_Micro, moketa:U_PRO_MICRO

Commit message: some fix
Parts:
- added D1: Diode, moketa:D_SOD-123, F.Cu at (173.7, 199.0)
- added D10: Diode, moketa:D_SOD-123, F.Cu at (179.5, 199.0)
- added D11: Diode, moketa:D_SOD-123, F.Cu at (179.5, 202.4)
- added D12: Diode, moketa:D_SOD-123, F.Cu at (179.5, 205.8)
- added D13: Diode, moketa:D_SOD-123, F.Cu at (179.5, 209.2)
- added D14: Diode, moketa:D_SOD-123, F.Cu at (179.5, 212.6)
- added D15: Diode, moketa:D_SOD-123, F.Cu at (179.5, 216.0)
- added D16: Diode, moketa:D_SOD-123, F.Cu at (179.5, 219.4)
- added D17: Diode, moketa:D_SOD-123, F.Cu at (179.5, 222.8)
- added D18: Diode, moketa:D_SOD-123, F.Cu at (179.5, 226.2)
- added D19: Diode, moketa:D_SOD-123, F.Cu at (185.3, 199.0)
- added D2: Diode, moketa:D_SOD-123, F.Cu at (173.7, 202.4)
- added D20: Diode, moketa:D_SOD-123, F.Cu at (185.3, 202.4)
- added D21: Diode, moketa:D_SOD-123, F.Cu at (185.3, 205.8)
- added D22: Diode, moketa:D_SOD-123, F.Cu at (185.3, 209.2)
- added D23: Diode, moketa:D_SOD-123, F.Cu at (185.3, 212.6)
- added D24: Diode, moketa:D_SOD-123, F.Cu at (185.3, 216.0)
- added D25: Diode, moketa:D_SOD-123, F.Cu at (185.3, 219.4)
- added D26: Diode, moketa:D_SOD-123, F.Cu at (185.3, 222.8)
- added D27: Diode, moketa:D_SOD-123, F.Cu at (185.3, 226.2)
- added D28: Diode, moketa:D_SOD-123, F.Cu at (191.1, 199.0)
- added D29: Diode, moketa:D_SOD-123, F.Cu at (191.1, 202.4)
- added D3: Diode, moketa:D_SOD-123, F.Cu at (173.7, 205.8)
- added D30: Diode, moketa:D_SOD-123, F.Cu at (191.1, 205.8)
- added D31: Diode, moketa:D_SOD-123, F.Cu at (191.1, 209.2)
- added D32: Diode, moketa:D_SOD-123, F.Cu at (191.1, 212.6)
- added D33: Diode, moketa:D_SOD-123, F.Cu at (191.1, 216.0)
- added D34: Diode, moketa:D_SOD-123, F.Cu at (191.1, 219.4)
- added D35: Diode, moketa:D_SOD-123, F.Cu at (191.1, 222.8)
- added D36: Diode, moketa:D_SOD-123, F.Cu at (191.1, 226.2)
- added D37: Diode, moketa:D_SOD-123, F.Cu at (196.9, 199.0)
- added D38: Diode, moketa:D_SOD-123, F.Cu at (196.9, 202.4)
- added D39: Diode, moketa:D_SOD-123, F.Cu at (196.9, 205.8)
- added D4: Diode, moketa:D_SOD-123, F.Cu at (173.7, 209.2)
- added D40: Diode, moketa:D_SOD-123, F.Cu at (196.9, 209.2)
- added D41: Diode, moketa:D_SOD-123, F.Cu at (196.9, 212.6)
- added D42: Diode, moketa:D_SOD-123, F.Cu at (196.9, 216.0)
- added D5: Diode, moketa:D_SOD-123, F.Cu at (173.7, 212.6)
- added D6: Diode, moketa:D_SOD-123, F.Cu at (173.7, 216.0)
- added D7: Diode, moketa:D_SOD-123, F.Cu at (173.7, 219.4)
- added D8: Diode, moketa:D_SOD-123, F.Cu at (173.7, 222.8)
- added D9: Diode, moketa:D_SOD-123, F.Cu at (173.7, 226.2)
- added J1: ~, moketa:J_BATTERY, F.Cu at (174.7, 229.3)
- added LED1: ~, moketa:YS-SK6812MINI-E, F.Cu at (117.8, 199.3)
- added LED10: ~, moketa:YS-SK6812MINI-E, F.Cu at (125.3, 199.3)
- added LED11: ~, moketa:YS-SK6812MINI-E, F.Cu at (125.3, 203.3)
- added LED12: ~, moketa:YS-SK6812MINI-E, F.Cu at (125.3, 207.3)
- added LED13: ~, moketa:YS-SK6812MINI-E, F.Cu at (125.3, 211.3)
- added LED14: ~, moketa:YS-SK6812MINI-E, F.Cu at (125.3, 215.3)
- added LED15: ~, moketa:YS-SK6812MINI-E, F.Cu at (125.3, 219.3)
- added LED16: ~, moketa:YS-SK6812MINI-E, F.Cu at (125.3, 223.3)
- added LED17: ~, moketa:YS-SK6812MINI-E, F.Cu at (125.3, 227.3)
- added LED18: ~, moketa:YS-SK6812MINI-E, F.Cu at (125.3, 231.3)
- added LED19: ~, moketa:YS-SK6812MINI-E, F.Cu at (132.9, 199.3)
- added LED2: ~, moketa:YS-SK6812MINI-E, F.Cu at (117.8, 203.3)
- added LED20: ~, moketa:YS-SK6812MINI-E, F.Cu at (132.9, 203.3)
- added LED21: ~, moketa:YS-SK6812MINI-E, F.Cu at (132.9, 207.3)
- added LED22: ~, moketa:YS-SK6812MINI-E, F.Cu at (132.9, 211.3)
- added LED23: ~, moketa:YS-SK6812MINI-E, F.Cu at (132.9, 215.3)
- added LED24: ~, moketa:YS-SK6812MINI-E, F.Cu at (132.9, 219.3)
- added LED25: ~, moketa:YS-SK6812MINI-E, F.Cu at (132.9, 223.3)
- added LED26: ~, moketa:YS-SK6812MINI-E, F.Cu at (132.9, 227.3)
- added LED27: ~, moketa:YS-SK6812MINI-E, F.Cu at (132.9, 231.3)
- added LED28: ~, moketa:YS-SK6812MINI-E, F.Cu at (140.5, 199.3)
- added LED29: ~, moketa:YS-SK6812MINI-E, F.Cu at (140.5, 203.3)
- added LED3: ~, moketa:YS-SK6812MINI-E, F.Cu at (117.8, 207.3)
- added LED30: ~, moketa:YS-SK6812MINI-E, F.Cu at (140.5, 207.3)
- added LED31: ~, moketa:YS-SK6812MINI-E, F.Cu at (140.5, 211.3)
- added LED32: ~, moketa:YS-SK6812MINI-E, F.Cu at (140.5, 215.3)
- added LED33: ~, moketa:YS-SK6812MINI-E, F.Cu at (140.5, 219.3)
- added LED34: ~, moketa:YS-SK6812MINI-E, F.Cu at (140.5, 223.3)
- added LED35: ~, moketa:YS-SK6812MINI-E, F.Cu at (140.5, 227.3)
- added LED36: ~, moketa:YS-SK6812MINI-E, F.Cu at (140.5, 231.3)
- added LED37: ~, moketa:YS-SK6812MINI-E, F.Cu at (148.1, 199.3)
- added LED38: ~, moketa:YS-SK6812MINI-E, F.Cu at (148.1, 203.3)
- added LED39: ~, moketa:YS-SK6812MINI-E, F.Cu at (148.1, 207.3)
- added LED4: ~, moketa:YS-SK6812MINI-E, F.Cu at (117.8, 211.3)
- added LED40: ~, moketa:YS-SK6812MINI-E, F.Cu at (148.1, 211.3)
- added LED41: ~, moketa:YS-SK6812MINI-E, F.Cu at (148.1, 215.3)
- added LED42: ~, moketa:YS-SK6812MINI-E, F.Cu at (148.1, 219.3)
- added LED5: ~, moketa:YS-SK6812MINI-E, F.Cu at (117.8, 215.3)
- added LED6: ~, moketa:YS-SK6812MINI-E, F.Cu at (117.8, 219.3)
- added LED7: ~, moketa:YS-SK6812MINI-E, F.Cu at (117.8, 223.3)
- added LED8: ~, moketa:YS-SK6812MINI-E, F.Cu at (117.8, 227.3)
- added LED9: ~, moketa:YS-SK6812MINI-E, F.Cu at (117.8, 231.3)
- added SW1: ~, moketa:SW_PUSH, F.Cu at (124.1, 86.8)
- added SW10: ~, moketa:SW_PUSH, F.Cu at (144.2, 147.1)
- added SW11: ~, moketa:SW_PUSH, F.Cu at (144.2, 167.2)
- added SW12: ~, moketa:SW_PUSH, F.Cu at (144.2, 187.3)
- added SW13: ~, moketa:SW_PUSH, F.Cu at (164.3, 86.8)
- added SW14: ~, moketa:SW_PUSH, F.Cu at (164.3, 106.9)
- added SW15: ~, moketa:SW_PUSH, F.Cu at (164.3, 127.0)
- added SW16: ~, moketa:SW_PUSH, F.Cu at (164.3, 147.1)
- added SW17: ~, moketa:SW_PUSH, F.Cu at (164.3, 167.2)
- added SW18: ~, moketa:SW_PUSH, F.Cu at (164.3, 187.3)
- added SW19: ~, moketa:SW_PUSH, F.Cu at (184.4, 86.8)
- added SW2: ~, moketa:SW_PUSH, F.Cu at (124.1, 106.9)
- added SW20: ~, moketa:SW_PUSH, F.Cu at (184.4, 106.9)
- added SW21: ~, moketa:SW_PUSH, F.Cu at (184.4, 127.0)
- added SW22: ~, moketa:SW_PUSH, F.Cu at (184.4, 147.1)
- added SW23: ~, moketa:SW_PUSH, F.Cu at (184.4, 167.2)
- added SW24: ~, moketa:SW_PUSH, F.Cu at (184.4, 187.3)
- added SW25: ~, moketa:SW_PUSH, F.Cu at (204.5, 86.8)
- added SW26: ~, moketa:SW_PUSH, F.Cu at (204.5, 106.9)
- added SW27: ~, moketa:SW_PUSH, F.Cu at (204.5, 127.0)
- added SW28: ~, moketa:SW_PUSH, F.Cu at (204.5, 147.1)
- added SW29: ~, moketa:SW_PUSH, F.Cu at (204.5, 167.2)
- added SW3: ~, moketa:SW_PUSH, F.Cu at (124.1, 127.0)
- added SW30: ~, moketa:SW_PUSH, F.Cu at (204.5, 187.3)
- added SW31: ~, moketa:SW_PUSH, F.Cu at (224.6, 86.8)
- added SW32: ~, moketa:SW_PUSH, F.Cu at (224.6, 106.9)
- added SW33: ~, moketa:SW_PUSH, F.Cu at (224.6, 127.0)
- added SW34: ~, moketa:SW_PUSH, F.Cu at (224.6, 147.1)
- added SW35: ~, moketa:SW_PUSH, F.Cu at (224.6, 167.2)
- added SW36: ~, moketa:SW_PUSH, F.Cu at (224.6, 187.3)
- added SW37: ~, moketa:SW_PUSH, F.Cu at (244.7, 86.8)
- added SW38: ~, moketa:SW_PUSH, F.Cu at (244.7, 106.9)
- added SW39: ~, moketa:SW_PUSH, F.Cu at (244.7, 127.0)
- added SW4: ~, moketa:SW_PUSH, F.Cu at (124.1, 147.1)
- added SW40: ~, moketa:SW_PUSH, F.Cu at (244.7, 147.1)
- added SW41: ~, moketa:SW_PUSH, F.Cu at (244.7, 167.2)
- added SW42: ~, moketa:SW_PUSH, F.Cu at (244.7, 187.3)
- added SW43: Reset, moketa:SW_TACT, F.Cu at (183.9, 229.3)
- added SW5: ~, moketa:SW_PUSH, F.Cu at (124.1, 167.2)
- added SW6: ~, moketa:SW_PUSH, F.Cu at (124.1, 187.3)
- added SW7: ~, moketa:SW_PUSH, F.Cu at (144.2, 86.8)
- added SW8: ~, moketa:SW_PUSH, F.Cu at (144.2, 106.9)
- added SW9: ~, moketa:SW_PUSH, F.Cu at (144.2, 127.0)
- added U1: Pro_Micro, moketa:U_PRO_MICRO, F.Cu at (161.3, 214.7)
Other:
- board outline added: 144.9 x 166.3 mm
